Commit message: Update my_robot.xacro

File: src/my_robot/urdf/my_robot.xacro (robot description, xacro)
@@ -8,4 +8,11 @@
     <child link="chassis" />
   </joint>
+  <joint name="camera_optical_joint" type="fixed">
+    <origin xyz="0 0 0" rpy="-1.5707 0 -1.5707"/>
+    <parent link="camera_link"/>
+    <child link="camera_link_optical"/>
+  </joint>
+  <link name="camera_link_optical">
+  </link>
   <link name='chassis'>
     <pose>0 0 0.1 0 0 0</pose>

Commit message: Changes

File: src/my_robot/urdf/my_robot.xacro (robot description, xacro)
@@ -3,4 +3,5 @@
   <xacro:include filename="$(find my_robot)/urdf/my_robot.gazebo" />
   <link name="robot_footprint"></link>
+  <link name="camera_link_optical" />
   <joint name="robot_footprint_joint" type="fixed">
     <origin xyz="0 0 0" rpy="0 0 0" />
@@ -13,6 +14,4 @@
     <child link="camera_link_optical"/>
   </joint>
-  <link name="camera_link_optical">
-  </link>
   <link name='chassis'>
     <pose>0 0 0.1 0 0 0</pose>

Commit message: Fixes

File: src/my_robot/urdf/my_robot.xacro (robot description, xacro)
@@ -3,5 +3,4 @@
   <xacro:include filename="$(find my_robot)/urdf/my_robot.gazebo" />
   <link name="robot_footprint"></link>
-  <link name="camera_link_optical" />
   <joint name="robot_footprint_joint" type="fixed">
     <origin xyz="0 0 0" rpy="0 0 0" />
@@ -14,4 +13,5 @@
     <child link="camera_link_optical"/>
   </joint>
+  <link name="camera_link_optical"></link>
   <link name='chassis'>
     <pose>0 0 0.1 0 0 0</pose>

Commit message: Changes

File: src/my_robot/urdf/my_robot.xacro (robot description, xacro)
@@ -10,5 +10,5 @@
   <joint name="camera_optical_joint" type="fixed">
     <origin xyz="0 0 0" rpy="-1.5707 0 -1.5707"/>
-    <parent link="camera_link"/>
+    <parent link="camera"/>
     <child link="camera_link_optical"/>
   </joint>
